Commit message: added models

File: install/artist_robot/share/artist_robot/urdf/artist_robot.urdf (robot description, URDF)
Before this commit: robot artist_robot, 12 links, 11 joints
Links:
- link base_link: geometry collision box size=0.5 0.3 0.1; visual box size=0.5 0.3 0.1
- link brush_arm: geometry collision box size=0.05 0.05 0.1; visual box size=0.05 0.05 0.1
- link brush_platform: geometry collision box size=0.2 0.2 0.02; visual box size=0.2 0.2 0.02
- link brush_tip: geometry collision cylinder length=0.05 radius=0.01; visual cylinder length=0.05 radius=0.01
- link brush_tip_extension: geometry collision cylinder length=0.05 radius=0.008; visual cylinder length=0.05 radius=0.008
- link lift_arm: geometry collision cylinder length=0.5 radius=0.03; visual cylinder length=0.5 radius=0.03
- link wheel_1: geometry collision cylinder length=0.02 radius=0.05; visual cylinder length=0.02 radius=0.05
- link wheel_2: geometry collision cylinder length=0.02 radius=0.05; visual cylinder length=0.02 radius=0.05
- link wheel_3: geometry collision cylinder length=0.02 radius=0.05; visual cylinder length=0.02 radius=0.05
- link wheel_4: geometry collision cylinder length=0.02 radius=0.05; visual cylinder length=0.02 radius=0.05
Joints:
- joint base_to_lift_arm: origin xyz=0 0 0.05 rpy=0 0 0 -> xyz=0 0 0.06 rpy=0 0 0
- joint brush_tip_to_extension: limit lower=0 upper=0.11 effort=10 velocity=0.1 -> lower=0 upper=0.1 effort=10 velocity=0.1
- joint lift_arm_to_brush_platform: origin xyz=0 0 0.05 -> xyz=0 0 0.5
