Commit message: modified urdf

File: urdf/artist_robot.urdf (robot description, URDF)
Before this commit: robot artist_robot, 11 links, 10 joints
Links:
- added link lift_arm, mass 0.5; collision cylinder length=0.1 radius=0.05; visual cylinder length=0.1 radius=0.05
Joints:
- removed joint base_to_brush_platform
- added joint base_to_lift_arm: type prismatic, parent base_link, child lift_arm, origin xyz=0 0 0.05 rpy=0 0 0, axis 0 0 1, limit lower=0 upper=0.5 effort=20 velocity=0.2
- added joint lift_arm_to_brush_platform: type fixed, parent lift_arm, child brush_platform, origin xyz=0 0 0.05

Commit message: gazebo beggining

File: urdf/artist_robot.urdf (robot description, URDF)
Before this commit: robot artist_robot, 12 links, 11 joints
Links:
- link base_link: geometry collision box size=0.5 0.3 0.1; visual mesh filename=file://$(find artist_robot)/urdf/base_link.dae
- link brush_arm: geometry collision box size=0.05 0.05 0.1; visual mesh filename=file://$(find artist_robot)/urdf/brush_arm.dae
- link brush_platform: geometry collision box size=0.2 0.2 0.02; visual mesh filename=file://$(find artist_robot)/urdf/brush_platform.dae
- link brush_tip: geometry collision cylinder length=0.05 radius=0.01; visual mesh filename=file://$(find artist_robot)/urdf/brush_tip.dae
- link brush_tip_extension: geometry collision cylinder length=0.05 radius=0.008; visual mesh filename=file://$(find artist_robot)/urdf/brush_tip_extension.dae
- link lift_arm: geometry collision cylinder length=0.1 radius=0.05; visual mesh filename=file://$(find artist_robot)/urdf/lift_arm.dae
- link wheel_1: geometry collision cylinder length=0.02 radius=0.05; visual mesh filename=file://$(find artist_robot)/urdf/wheel.dae
- link wheel_2: geometry collision cylinder length=0.02 radius=0.05; visual mesh filename=file://$(find artist_robot)/urdf/wheel.dae
- link wheel_3: geometry collision cylinder length=0.02 radius=0.05; visual mesh filename=file://$(find artist_robot)/urdf/wheel.dae
- link wheel_4: geometry collision cylinder length=0.02 radius=0.05; visual mesh filename=file://$(find artist_robot)/urdf/wheel.dae
Joints:
- joint brush_tip_to_extension: limit lower=0 upper=0.11 effort=10 velocity=0.1 -> lower=0 upper=0.25 effort=10 velocity=0.1
- joint platform_to_brush_arm: axis 0 0 1 -> 1 0 0; type planar -> prismatic

Commit message: Update artist_robot.urdf

File: urdf/artist_robot.urdf (robot description, URDF)
Before this commit: robot artist_robot, 12 links, 11 joints
Links:
- removed link wheel_1
- removed link wheel_2
- removed link wheel_3
- removed link wheel_4
- removed link wheel_mount_1
- removed link wheel_mount_2
- added link caster_wheel, mass 0.5; collision sphere radius=0.035; visual sphere radius=0.035
- added link left_wheel, mass 0.5; collision cylinder length=0.02 radius=0.05; visual cylinder length=0.02 radius=0.05
- added link right_wheel, mass 0.5; collision cylinder length=0.02 radius=0.05; visual cylinder length=0.02 radius=0.05
- link base_link: geometry collision box size=0.5 0.3 0.1; visual box size=0.5 0.3 0.1
- link brush_arm: geometry collision box size=0.05 0.05 0.1; visual box size=0.05 0.05 0.1
- link brush_platform: geometry collision box size=0.2 0.2 0.02; visual box size=0.2 0.2 0.02
- link brush_tip: geometry collision cylinder length=0.05 radius=0.01; visual cylinder length=0.05 radius=0.01
- link brush_tip_extension: geometry collision cylinder length=0.05 radius=0.008; visual cylinder length=0.05 radius=0.008
- link lift_arm: geometry collision cylinder length=0.1 radius=0.05; visual cylinder length=0.1 radius=0.05
Joints:
- removed joint base_to_wheel_3
- removed joint base_to_wheel_4
- removed joint base_to_wheel_mount_1
- removed joint base_to_wheel_mount_2
- removed joint mount_1_to_wheel_1
- removed joint mount_2_to_wheel_2
- added joint base_to_caster_wheel: type fixed, parent base_link, child caster_wheel, origin xyz=-0.2 0.0 -0.06 rpy=0 0 0
- added joint base_to_left_wheel: type continuous, parent base_link, child left_wheel, origin xyz=0.2 0.15 -0.05 rpy=1.5708 0 0, axis 0 0 1
- added joint base_to_right_wheel: type continuous, parent base_link, child right_wheel, origin xyz=0.2 -0.15 -0.05 rpy=1.5708 0 0, axis 0 0 1
